File: Bat Listener Hardware/Bat_Listner_JLCPCB/Bat_Listner_JLCPCB.sch (KiCad schematic (older format))
At the start: 29 parts

Commit message: Finished schematic
Parts:
- removed IC?: CD4042BDR, SOIC127P600X175-16N, symbol Digital_JLC:CD4042BDR
- added C14: 100u_T, SamacSys_Parts:CAPPM3528X210N, symbol Capacitor_JLC:100u_T
- added C4: 220uF_E, Capacitor_SMD:CP_Elec_6.3x7.7, symbol Capacitor_JLC:220uF_E
- added C5: 47n, Capacitor_SMD:C_0402_1005Metric, symbol Capacitor_JLC:47n
- added D1: ZMM5V1, Diode_SMD:D_MiniMELF, symbol Diode_JLC:ZMM5V1
- added D4: RedLED, Diode_SMD:D_0805_2012Metric, symbol Diode_JLC:RedLED
- added IC1: CD4024BM96, SamacSys_Parts:SOIC127P600X175-14N, symbol Digital_JLC:CD4024BM96
- added IC2: TL074IDR, SamacSys_Parts:SOIC127P600X175-14N, symbol Transistor_JLC:TL074IDR
- added J1, J2, J3, J5: B2B-PH-K-S_LF__SN_, SamacSys_Parts:SHDR2W50P0X200_1X2_590X450X600P, symbol SamacSys_Parts:B2B-PH-K-S_LF__SN_
- added J6: STX-3200-3NB, SamacSys_Parts:STX32003NB, symbol SamacSys_Parts:STX-3200-3NB
- added JP1: SolderJumper_2_Bridged, Jumper:SolderJumper-2_P1.3mm_Bridged_Pad1.0x1.5mm, symbol Jumper:SolderJumper_2_Bridged
- added JP2: SolderJumper_2_Open, Jumper:SolderJumper-2_P1.3mm_Open_Pad1.0x1.5mm, symbol Jumper:SolderJumper_2_Open
- added R11: 100, Resistor_SMD:R_0402_1005Metric, symbol Resistor_JLC:100
- added RV1, RV2: 22k, Potentiometer_THT:Potentiometer_Bourns_3296W_Vertical, symbol Device:R_POT
- AT1: renamed from AT?; footprint SOIC127P600X175-8N -> SamacSys_Parts:SOIC127P600X175-8N
- Q1: renamed from Q?; footprint SOT65P210X110-3N -> SamacSys_Parts:SOT65P210X110-3N
- gave numbers to parts that had none: 26
Connections:
- net at AT1.1 (GAIN_1): now also C1.2
- net at AT1.2 (-INPUT): now also J1.1
- net at AT1.3 (+INPUT): now also J1.2
- net GND: now reaches AT1.4 (GND)
- net GND: now also C2.2, C3.2, D2.2 (A), Q1.2, R4.2, R5.2, R7.2, C14.2, C4.2, C5.2, D1.2 (A), IC1.2 (RESET), IC1.7 (VSS), J2.2
- net at AT1.5 (VOUT): now also C6.1, R2.1
- net +BATT: now reaches AT1.6 (VS)
- net +BATT: now also R9.1, C4.1, C5.1, IC1.14 (VDD)
- net at AT1.7 (BYPASS): now also C2.1
- net at AT1.8 (GAIN_2): now also C1.1
- net at C3.1: now also R2.2
- net at C6.2: now also C8.2, C9.1, R4.1
- net 6: now reaches C8.1
- net 6: now also R6.2, IC2.6 (2IN-)
- net 7: now reaches C9.2
- net 7: now also C10.1, R6.1, IC2.7 (2OUT)
- net at C10.2: now also C11.1, C12.1, R7.1
- net 9: now reaches C11.2
- net 9: now also R8.1, IC2.9 (3IN-)
- net 8: now reaches C12.2
- net 8: now also C13.1, R8.2, IC2.8 (3OUT)
- net at C13.2: now also RV2.3
- net 14: now reaches R12.1
- net 14: now also C15.2, IC1.1 ([Oslash]), IC2.14 (4OUT)
- net 13: now reaches R12.2
- net 13: now also C15.1, IC2.13 (4IN-), RV2.1, RV2.2
- net at Q1.1: now also C7.2, D2.1 (K), R5.1
- net at Q1.3: now also D3.2 (A), R10.2, D4.1 (K), J3.2, JP2.2 (B)
- net at R3.1: now also R1.1, IC1.6 (Q4)
- net at R3.2: now also C7.1
- net at R1.2: now also D1.1 (K), J2.1
- net at D3.1 (K): now also R10.1, R9.2, C14.1, D4.2 (A), J3.1, J5.1, RV1.3
- net at C16.1: now also J6.2 (2R), J6.3 (5T), R11.2
- net at C16.2: now also J5.2, JP1.1 (A)
- new net: R11.1, RV1.2
- new net: J6.1 (1S), JP1.2 (B), JP2.1 (A)
- new net GNDA: IC2.10 (3IN+), IC2.12 (4IN+), IC2.5 (2IN+)
- no-connect marks 0 -> 7
Other:
- moved on the sheet: AT1, C1, C10, C11, C12, C13, C15, C16, C2, C3, C6, C7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

Commit message: prelim layout with TPs
Parts:
- added J4: B2B-PH-K-S_LF__SN_, SamacSys_Parts:SHDR2W50P0X200_1X2_590X450X600P, symbol SamacSys_Parts:B2B-PH-K-S_LF__SN_
- added TP1, TP2, TP3, TP4, TP5, TP6, TP7: TestPoint, TestPoint:TestPoint_Keystone_5000-5004_Miniature, symbol personal:TestPoint
Connections:
- net +BATT: now also J4.1, TP4.1
- net 14: now also TP7.1
- net 7: now also TP5.1
- net 8: now also TP6.1
- net GND: now also J4.2, TP3.1
- net at AT1.2 (-INPUT), J1.1: now also TP1.1
- net at AT1.3 (+INPUT), J1.2: now also TP2.1
Changed lines of the file:
@@
 $EndComp
 Wire Wire Line
-	2400 3700 2950 3700
-Wire Wire Line
-	2400 3800 2950 3800
+	2400 3700 2450 3700
+Wire Wire Line
+	2400 3800 2450 3800
 $Comp
 L power:GND #PWR0101
@@
 Wire Wire Line
 	4550 3800 4550 3000
-Wire Wire Line
-	4550 3000 4700 3000
 $Comp
 L Capacitor_JLC:220uF_E C4
@@
 $EndComp
 Wire Wire Line
-	4700 3000 4700 3100
+	4700 3000 4700 3050
 Connection ~ 4700 3000
 $Comp
@@
 8
 Wire Wire Line
-	9150 3850 9150 4350
-Wire Wire Line
 	9150 4350 9050 4350
 Connection ~ 9150 3850
@@
 Wire Wire Line
 	10900 4050 11100 4050
-Wire Wire Line
-	11100 4050 11100 3600
 Wire Wire Line
 	11100 3250 10700 3250
@@
 Wire Wire Line
 	9650 7300 12450 7300
+$Comp
+L personal:TestPoint TP4
+U 1 1 5FF01E2C
+P 4800 3050
+F 0 "TP4" H 5060 3144 50  0000 L CNN
+F 1 "TestPoint" H 5060 3053 50  0000 L CNN
+F 2 "TestPoint:TestPoint_Keystone_5000-5004_Miniature" H 5000 3050 50  0001 C CNN
+F 3 "~" H 5000 3050 50  0001 C CNN
+	1    4800 3050
+	1    0    0    -1
+$EndComp
+Wire Wire Line
+	4800 3050 4700 3050
+Connection ~ 4700 3050
+Wire Wire Line
+	4700 3050 4700 3100
+$Comp
+L personal:TestPoint TP1
+U 1 1 5FF0C4B2
+P 2450 3700
+F 0 "TP1" H 2600 3850 50  0000 L CNN
+F 1 "TestPoint" H 2600 3950 50  0000 L CNN
+F 2 "TestPoint:TestPoint_Keystone_5000-5004_Miniature" H 2650 3700 50  0001 C CNN
+F 3 "~" H 2650 3700 50  0001 C CNN
+	1    2450 3700
+	1    0    0    -1
+$EndComp
+Connection ~ 2450 3700
+Wire Wire Line
+	2450 3700 2950 3700
+$Comp
+L personal:TestPoint TP2
+U 1 1 5FF0D234
+P 2450 3800
+F 0 "TP2" H 2600 3950 50  0000 R CNN
+F 1 "TestPoint" H 2700 4050 50  0000 R CNN
+F 2 "TestPoint:TestPoint_Keystone_5000-5004_Miniature" H 2650 3800 50  0001 C CNN
+F 3 "~" H 2650 3800 50  0001 C CNN
+	1    2450 3800
+	1    0    0    1
+$EndComp
+Connection ~ 2450 3800
+Wire Wire Line
+	2450 3800 2950 3800
+$Comp
+L personal:TestPoint TP7
+U 1 1 5FF0DC1A
+P 11100 3250
+F 0 "TP7" H 11360 3344 50  0000 L CNN
+F 1 "TestPoint" H 11360 3253 50  0000 L CNN
+F 2 "TestPoint:TestPoint_Keystone_5000-5004_Miniature" H 11300 3250 50  0001 C CNN
+F 3 "~" H 11300 3250 50  0001 C CNN
+	1    11100 3250
+	1    0    0    -1
+$EndComp
+$Comp
+L personal:TestPoint TP6
+U 1 1 5FF0E32B
+P 9150 3450
+F 0 "TP6" H 9410 3544 50  0000 L CNN
+F 1 "TestPoint" H 9410 3453 50  0000 L CNN
+F 2 "TestPoint:TestPoint_Keystone_5000-5004_Miniature" H 9350 3450 50  0001 C CNN
+F 3 "~" H 9350 3450 50  0001 C CNN
+	1    9150 3450
+	1    0    0    -1
+$EndComp
+$Comp
+L personal:TestPoint TP5
+U 1 1 5FF1FD7C
+P 7350 3450
+F 0 "TP5" H 7610 3544 50  0000 L CNN
+F 1 "TestPoint" H 7610 3453 50  0000 L CNN
+F 2 "TestPoint:TestPoint_Keystone_5000-5004_Miniature" H 7550 3450 50  0001 C CNN
+F 3 "~" H 7550 3450 50  0001 C CNN
+	1    7350 3450
+	1    0    0    -1
+$EndComp
+Connection ~ 7350 3450
+Connection ~ 9150 3450
+Connection ~ 11100 3250
+Wire Wire Line
+	11100 3600 11100 4050
+Wire Wire Line
+	9150 3850 9150 4350
+$Comp
+L personal:TestPoint TP3
+U 1 1 5FF212F5
+P 3750 8750
+F 0 "TP3" H 3900 8950 50  0000 R CNN
+F 1 "TestPoint" H 4100 9050 50  0000 R CNN
+F 2 "TestPoint:TestPoint_Keystone_5000-5004_Miniature" H 3950 8750 50  0001 C CNN
+F 3 "~" H 3950 8750 50  0001 C CNN
+	1    3750 8750
+	-1   0    0    1
+$EndComp
+Connection ~ 3750 8750
+$Comp
+L SamacSys_Parts:B2B-PH-K-S_LF__SN_ J4
+U 1 1 5FF830D7
+P 6000 2200
+F 0 "J4" H 6292 2465 50  0000 C CNN
+F 1 "B2B-PH-K-S_LF__SN_" H 6292 2374 50  0000 C CNN
+F 2 "SamacSys_Parts:SHDR2W50P0X200_1X2_590X450X600P" H 6650 2300 50  0001 L CNN
+F 3 "http://www.jst-mfg.com/product/pdf/eng/ePH.pdf" H 6650 2200 50  0001 L CNN
+F 4 "PH-2.0mm Header top entry 2 way JST PH Series, Series Number B2B, 2mm Pitch 2 Way 1 Row Straight PCB Header, Through Hole Termination, 2A" H 6650 2100 50  0001 L CNN "Description"
+F 5 "6" H 6650 2000 50  0001 L CNN "Height"
+F 6 "JST (JAPAN SOLDERLESS TERMINALS)" H 6650 1900 50  0001 L CNN "Manufacturer_Name"
+F 7 "B2B-PH-K-S(LF)(SN)" H 6650 1800 50  0001 L CNN "Manufacturer_Part_Number"
+F 8 "8201422P" H 6650 1500 50  0001 L CNN "RS Part Number"
+F 9 "http://uk.rs-online.com/web/p/products/8201422P" H 6650 1400 50  0001 L CNN "RS Price/Stock"
+	1    6000 2200
+	1    0    0    -1
+$EndComp
+Wire Wire Line
+	4550 3000 4700 3000
+Wire Wire Line
+	6000 2200 4550 2200
+Wire Wire Line
+	4550 2200 4550 3000
+Connection ~ 4550 3000
+Wire Wire Line
+	4700 3350 6000 3350
+Wire Wire Line
+	6000 3350 6000 2300
+Connection ~ 4700 3350
 $EndSCHEMATC

Commit message: finished layout
Parts:
- removed J1: B2B-PH-K-S_LF__SN_, SamacSys_Parts:SHDR2W50P0X200_1X2_590X450X600P, symbol SamacSys_Parts:B2B-PH-K-S_LF__SN_
- removed TP1, TP2, TP5, TP6, TP7: TestPoint, TestPoint:TestPoint_Keystone_5000-5004_Miniature, symbol personal:TestPoint
- added IC3: MA40S4S, MA40S4S, symbol SamacSys_Parts:MA40S4S
- renumbered TP4 to TP1, TP3 to TP2
Connections:
- net at AT1.2 (-INPUT): now also IC3.1
- net at AT1.3 (+INPUT): now also IC3.2
Changed lines of the file:
@@
 $EndComp
-$Comp
-L SamacSys_Parts:B2B-PH-K-S_LF__SN_ J1
-U 1 1 5FE892ED
-P 2400 3700
-F 0 "J1" H 2692 3965 50  0000 C CNN
-F 1 "B2B-PH-K-S_LF__SN_" H 2692 3874 50  0000 C CNN
-F 2 "SamacSys_Parts:SHDR2W50P0X200_1X2_590X450X600P" H 3050 3800 50  0001 L CNN
-F 3 "http://www.jst-mfg.com/product/pdf/eng/ePH.pdf" H 3050 3700 50  0001 L CNN
-F 4 "PH-2.0mm Header top entry 2 way JST PH Series, Series Number B2B, 2mm Pitch 2 Way 1 Row Straight PCB Header, Through Hole Termination, 2A" H 3050 3600 50  0001 L CNN "Description"
-F 5 "6" H 3050 3500 50  0001 L CNN "Height"
-F 6 "JST (JAPAN SOLDERLESS TERMINALS)" H 3050 3400 50  0001 L CNN "Manufacturer_Name"
-F 7 "B2B-PH-K-S(LF)(SN)" H 3050 3300 50  0001 L CNN "Manufacturer_Part_Number"
-F 8 "8201422P" H 3050 3000 50  0001 L CNN "RS Part Number"
-F 9 "http://uk.rs-online.com/web/p/products/8201422P" H 3050 2900 50  0001 L CNN "RS Price/Stock"
-	1    2400 3700
-	-1   0    0    -1
-$EndComp
-Wire Wire Line
-	2400 3700 2450 3700
-Wire Wire Line
-	2400 3800 2450 3800
 $Comp
 L power:GND #PWR0101
@@
 Wire Wire Line
 	9650 7300 12450 7300
-$Comp
-L personal:TestPoint TP4
-U 1 1 5FF01E2C
-P 4800 3050
-F 0 "TP4" H 5060 3144 50  0000 L CNN
-F 1 "TestPoint" H 5060 3053 50  0000 L CNN
-F 2 "TestPoint:TestPoint_Keystone_5000-5004_Miniature" H 5000 3050 50  0001 C CNN
-F 3 "~" H 5000 3050 50  0001 C CNN
-	1    4800 3050
-	1    0    0    -1
-$EndComp
 Wire Wire Line
 	4800 3050 4700 3050
@@
 Wire Wire Line
 	4700 3050 4700 3100
-$Comp
-L personal:TestPoint TP1
-U 1 1 5FF0C4B2
-P 2450 3700
-F 0 "TP1" H 2600 3850 50  0000 L CNN
-F 1 "TestPoint" H 2600 3950 50  0000 L CNN
-F 2 "TestPoint:TestPoint_Keystone_5000-5004_Miniature" H 2650 3700 50  0001 C CNN
-F 3 "~" H 2650 3700 50  0001 C CNN
-	1    2450 3700
-	1    0    0    -1
-$EndComp
-Connection ~ 2450 3700
-Wire Wire Line
-	2450 3700 2950 3700
-$Comp
-L personal:TestPoint TP2
-U 1 1 5FF0D234
-P 2450 3800
-F 0 "TP2" H 2600 3950 50  0000 R CNN
-F 1 "TestPoint" H 2700 4050 50  0000 R CNN
-F 2 "TestPoint:TestPoint_Keystone_5000-5004_Miniature" H 2650 3800 50  0001 C CNN
-F 3 "~" H 2650 3800 50  0001 C CNN
-	1    2450 3800
-	1    0    0    1
-$EndComp
-Connection ~ 2450 3800
-Wire Wire Line
-	2450 3800 2950 3800
-$Comp
-L personal:TestPoint TP7
-U 1 1 5FF0DC1A
-P 11100 3250
-F 0 "TP7" H 11360 3344 50  0000 L CNN
-F 1 "TestPoint" H 11360 3253 50  0000 L CNN
-F 2 "TestPoint:TestPoint_Keystone_5000-5004_Miniature" H 11300 3250 50  0001 C CNN
-F 3 "~" H 11300 3250 50  0001 C CNN
-	1    11100 3250
-	1    0    0    -1
-$EndComp
-$Comp
-L personal:TestPoint TP6
-U 1 1 5FF0E32B
-P 9150 3450
-F 0 "TP6" H 9410 3544 50  0000 L CNN
-F 1 "TestPoint" H 9410 3453 50  0000 L CNN
-F 2 "TestPoint:TestPoint_Keystone_5000-5004_Miniature" H 9350 3450 50  0001 C CNN
-F 3 "~" H 9350 3450 50  0001 C CNN
-	1    9150 3450
-	1    0    0    -1
-$EndComp
-$Comp
-L personal:TestPoint TP5
-U 1 1 5FF1FD7C
-P 7350 3450
-F 0 "TP5" H 7610 3544 50  0000 L CNN
-F 1 "TestPoint" H 7610 3453 50  0000 L CNN
-F 2 "TestPoint:TestPoint_Keystone_5000-5004_Miniature" H 7550 3450 50  0001 C CNN
-F 3 "~" H 7550 3450 50  0001 C CNN
-	1    7350 3450
-	1    0    0    -1
-$EndComp
-Connection ~ 7350 3450
-Connection ~ 9150 3450
-Connection ~ 11100 3250
 Wire Wire Line
 	11100 3600 11100 4050
 Wire Wire Line
 	9150 3850 9150 4350
-$Comp
-L personal:TestPoint TP3
-U 1 1 5FF212F5
-P 3750 8750
-F 0 "TP3" H 3900 8950 50  0000 R CNN
-F 1 "TestPoint" H 4100 9050 50  0000 R CNN
-F 2 "TestPoint:TestPoint_Keystone_5000-5004_Miniature" H 3950 8750 50  0001 C CNN
-F 3 "~" H 3950 8750 50  0001 C CNN
-	1    3750 8750
-	-1   0    0    1
-$EndComp
-Connection ~ 3750 8750
 $Comp
 L SamacSys_Parts:B2B-PH-K-S_LF__SN_ J4
@@
 	6000 3350 6000 2300
 Connection ~ 4700 3350
+$Comp
+L SamacSys_Parts:MA40S4S IC3
+U 1 1 5FF4E107
+P 2400 3700
+F 0 "IC3" H 2692 3965 50  0000 C CNN
+F 1 "MA40S4S" H 2692 3874 50  0000 C CNN
+F 2 "MA40S4S" H 3050 3800 50  0001 L CNN
+F 3 "" H 3050 3700 50  0001 L CNN
+F 4 "Ultrasonic transducer transmitter,0.2-4m Murata 0.2  4 m Barrel Ultrasonic Proximity Sensor, PCB" H 3050 3600 50  0001 L CNN "Description"
+F 5 "" H 3050 3500 50  0001 L CNN "Height"
+F 6 "81-MA40S4S" H 3050 3400 50  0001 L CNN "Mouser Part Number"
+F 7 "https://www.mouser.co.uk/ProductDetail/Murata-Electronics/MA40S4S?qs=dyqxRLCA4pZUsZeqTN%2FO6A%3D%3D" H 3050 3300 50  0001 L CNN "Mouser Price/Stock"
+F 8 "Murata Electronics" H 3050 3200 50  0001 L CNN "Manufacturer_Name"
+F 9 "MA40S4S" H 3050 3100 50  0001 L CNN "Manufacturer_Part_Number"
+	1    2400 3700
+	-1   0    0    -1
+$EndComp
+Wire Wire Line
+	2400 3800 2950 3800
+Wire Wire Line
+	2400 3700 2950 3700
+$Comp
+L personal:TestPoint TP1
+U 1 1 5FF01E2C
+P 4800 3050
+F 0 "TP1" H 5060 3144 50  0000 L CNN
+F 1 "TestPoint" H 5060 3053 50  0000 L CNN
+F 2 "TestPoint:TestPoint_Keystone_5000-5004_Miniature" H 5000 3050 50  0001 C CNN
+F 3 "~" H 5000 3050 50  0001 C CNN
+	1    4800 3050
+	1    0    0    -1
+$EndComp
+Connection ~ 3750 8750
+$Comp
+L personal:TestPoint TP2
+U 1 1 5FF212F5
+P 3750 8750
+F 0 "TP2" H 3900 8950 50  0000 R CNN
+F 1 "TestPoint" H 4100 9050 50  0000 R CNN
+F 2 "TestPoint:TestPoint_Keystone_5000-5004_Miniature" H 3950 8750 50  0001 C CNN
+F 3 "~" H 3950 8750 50  0001 C CNN
+	1    3750 8750
+	-1   0    0    1
+$EndComp
 $EndSCHEMATC
