File: Bat Listener Hardware/Bat_Listner_JLCPCB/Bat_Listner_JLCPCB.kicad_pcb (KiCad board)
At the start: 2 copper layers, 45 parts, among them IC1 CD4024BM96, IC2 TL074IDR, J1 B2B-PH-K-S_LF__SN_, J2 B2B-PH-K-S_LF__SN_, J3 B2B-PH-K-S_LF__SN_, J5 B2B-PH-K-S_LF__SN_, J6 STX-3200-3NB, Q1 BC817-40W,115

Commit message: prelim layout with TPs
Parts:
- added J4: B2B-PH-K-S_LF__SN_, SamacSys_Parts:SHDR2W50P0X200_1X2_590X450X600P, F.Cu at (137.8, 82.5)
- added TP1: TestPoint, TestPoint:TestPoint_Keystone_5000-5004_Miniature, F.Cu at (99.5, 71.5)
- added TP2: TestPoint, TestPoint:TestPoint_Keystone_5000-5004_Miniature, F.Cu at (99.5, 75.9)
- added TP3: TestPoint, TestPoint:TestPoint_Keystone_5000-5004_Miniature, F.Cu at (103.8, 71.5)
- added TP4: TestPoint, TestPoint:TestPoint_Keystone_5000-5004_Miniature, F.Cu at (103.8, 75.9)
- added TP5: TestPoint, TestPoint:TestPoint_Keystone_5000-5004_Miniature, F.Cu at (108.2, 71.5)
- added TP6: TestPoint, TestPoint:TestPoint_Keystone_5000-5004_Miniature, F.Cu at (108.2, 75.9)
- added TP7: TestPoint, TestPoint:TestPoint_Keystone_5000-5004_Miniature, F.Cu at (112.5, 71.5)
- moved RV2 51.4 mm to (170.2, 55.9), turned to 90 degrees
- moved C1 47.8 mm to (145.6, 53.3), turned to 180 degrees
- moved R4 47.6 mm to (153.7, 59.2), turned to 90 degrees
- moved AT1 46.3 mm to (145.4, 57.1)
- moved C2 43.5 mm to (150.5, 54.6)
- moved C5 43.4 mm to (147.2, 61.6), turned to 180 degrees
- moved C9 42.9 mm to (153.0, 62.9), turned to 180 degrees
- moved J1 42.8 mm to (137.8, 55.9), turned to 90 degrees
- moved C6 42.3 mm to (150.5, 59.1)
- moved C3 42.1 mm to (153.7, 57.1), turned to 270 degrees
- moved R8 40.8 mm to (159.4, 64.8)
- moved C13 40.6 mm to (164.5, 62.9)
- moved C12 37.7 mm to (160.0, 67.3), turned to 90 degrees
- moved JP2 37.1 mm to (165.7, 66.0), turned to 90 degrees
- moved C8 36.6 mm to (153.0, 61.6), turned to 180 degrees
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
Commit message: finished layout
Parts:
- removed J1: B2B-PH-K-S_LF__SN_, SamacSys_Parts:SHDR2W50P0X200_1X2_590X450X600P
- removed the TP1 at (99.5, 71.5)
- removed the TP2 at (99.5, 75.9)
- removed TP5, TP6, TP7: TestPoint, TestPoint:TestPoint_Keystone_5000-5004_Miniature
- added IC3: MA40S4S, MA40S4S, F.Cu at (136.5, 61.6)
- moved TP2 37.5 mm to (141.0, 76.8)
- moved TP1 33.4 mm to (137.2, 76.8)
- moved R7 2.05 mm to (153.9, 66.8)
- moved R3 0.80 mm to (148.8, 72.9)
- moved C16 0.13 mm to (154.4, 77.0)
- renumbered TP4 to TP1, TP3 to TP2
Other:
- board outline added: 44.4 x 40.6 mm

Commit message: Finished PCB
Parts:
- turned C9 to 0 degrees
Routing:
- net GND: track 0.00 -> 109.1 mm, vias 0 -> 6
- net +BATT: track 0.00 -> 62.3 mm, vias 0 -> 1
- net Net-(C14-Pad1): track 0.00 -> 43.4 mm, vias 0 -> 2
- net Net-(J6-Pad1): track 0.00 -> 31.8 mm, vias 0 -> 1
- net Net-(C16-Pad1): track 0.00 -> 30.4 mm
- net Net-(D3-Pad2): track 0.00 -> 24.5 mm, vias 0 -> 1
- net 14: track 0.00 -> 24.2 mm, vias 0 -> 2
- net Net-(C16-Pad2): track 0.00 -> 22.9 mm, vias 0 -> 2
- net 13: track 0.00 -> 10.9 mm
- net GNDA: track 0.00 -> 10.3 mm
- net Net-(AT1-Pad3): track 0.00 -> 9.60 mm
- net Net-(C10-Pad2): track 0.00 -> 8.78 mm
- net Net-(D1-Pad1): track 0.00 -> 8.42 mm
- net Net-(R11-Pad1): track 0.00 -> 8.08 mm
- net 9: track 0.00 -> 7.91 mm
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Other:
- net class Default: trace_width 0.25 -> 0.15; via_dia 0.8 -> 0.4; via_drill 0.4 -> 0.3
- rule trace_min: 0.2 -> 0.127
- rule via_min_size: 0.4 -> 0.3
