File: Bat_Listner_JLCPCB/Bat_Listner_JLCPCB.kicad_pcb (KiCad board)
At the start: 2 copper layers, 44.4 x 40.6 mm, 48 parts, among them IC1 CD4024BM96, IC2 TL074IDR, IC3 MA40S4S, J2 B2B-PH-K-S_LF__SN_, J3 B2B-PH-K-S_LF__SN_, J4 B2B-PH-K-S_LF__SN_, J5 B2B-PH-K-S_LF__SN_, J6 STX-3200-3NB, Q1 BC817-40W,115

Commit message: completed wiring
Parts:
- added C17: 100uF_E, Capacitor_SMD:CP_Elec_6.3x7.7, F.Cu at (161.8, 50.0)
- added C18: 100uF_E, Capacitor_SMD:CP_Elec_6.3x7.7, F.Cu at (144.3, 85.0)
- added R13: 68k, Resistor_SMD:R_0402_1005Metric, F.Cu at (155.2, 53.3)
- added R14: 68k, Resistor_SMD:R_0402_1005Metric, F.Cu at (156.5, 53.3)
- C4: value 220uF_E -> 100uF_E
- moved C4 34.4 mm to (150.4, 50.0), turned to 0 degrees
Connections:
- AT1 pad 4: GND -> 11
- AT1 pad 6: +BATT -> 4
- C14 pad 2: GND -> 11
- C2 pad 2: GND -> 11
- C3 pad 2: GND -> 11
- C4 pad 1: +BATT -> 4
- C4 pad 2: GND -> 3
- C5 pad 1: +BATT -> 4
- C5 pad 2: GND -> 11
- D1 pad 2: GND -> 11
- D2 pad 2: GND -> 11
- IC1 pad 14: +BATT -> 4
- IC1 pad 2: GND -> 11
- IC1 pad 7: GND -> 11
- IC2 pad 1: Net-(IC2-Pad1) -> 1
- IC2 pad 10: GNDA -> 1
- IC2 pad 11: Net-(IC2-Pad11) -> 11
- IC2 pad 12: GNDA -> 1
- IC2 pad 2: Net-(IC2-Pad2) -> 1
- IC2 pad 3: Net-(IC2-Pad3) -> 3
- IC2 pad 4: Net-(IC2-Pad4) -> 4
- IC2 pad 5: GNDA -> 1
- J2 pad 2: GND -> 11
- J4 pad 1: +BATT -> 4
- J4 pad 2: GND -> 11
- Q1 pad 2: GND -> 11
- R4 pad 2: GND -> 11
- R5 pad 2: GND -> 11
- R7 pad 2: GND -> 11
- R9 pad 1: +BATT -> 4
- TP1 pad 1: +BATT -> 4
- TP2 pad 1: GND -> 11
Routing:
- net 11: track 0.00 -> 143.0 mm, vias 0 -> 10
- net GND: track 109.1 -> 0.00 mm, vias 6 -> 0
- net 4: track 0.00 -> 89.7 mm, vias 0 -> 4
- net +BATT: track 62.3 -> 0.00 mm, vias 1 -> 0
- net 3: track 0.00 -> 20.3 mm, vias 0 -> 2
- net 1: track 0.00 -> 17.6 mm
- net GNDA: track 10.3 -> 0.00 mm
Other:
- board size 44.4 x 40.6 mm -> 44.2 x 47.2 mm
- board text added: "BAT LISTENER"
- board text added: "JT"

Commit message: updated pcb to fix audio jack
Parts:
- removed C16: 33n, Capacitor_SMD:C_0402_1005Metric
- removed J5: B2B-PH-K-S_LF__SN_, SamacSys_Parts:SHDR2W50P0X200_1X2_590X450X600P
- removed JP1: SolderJumper_2_Bridged, Jumper:SolderJumper-2_P1.3mm_Bridged_Pad1.0x1.5mm
- removed JP2: SolderJumper_2_Open, Jumper:SolderJumper-2_P1.3mm_Open_Pad1.0x1.5mm
Connections:
- net 4 renamed +BATT
- IC1 pad 10: Net-(IC1-Pad10) -> (no net)
- IC1 pad 11: Net-(IC1-Pad11) -> (no net)
- IC1 pad 12: Net-(IC1-Pad12) -> (no net)
- IC1 pad 13: Net-(IC1-Pad13) -> (no net)
- IC1 pad 3: Net-(IC1-Pad3) -> (no net)
- IC1 pad 4: Net-(IC1-Pad4) -> (no net)
- IC1 pad 5: Net-(IC1-Pad5) -> (no net)
- IC1 pad 8: Net-(IC1-Pad8) -> (no net)
- IC1 pad 9: Net-(IC1-Pad9) -> (no net)
- J6 pad 1: Net-(J6-Pad1) -> Net-(D3-Pad2)
- RV1 pad 1: Net-(RV1-Pad1) -> (no net)
Routing:
- net Net-(J6-Pad1): track 31.8 -> 0.00 mm, vias 1 -> 0
- net Net-(C16-Pad2): track 22.9 -> 0.00 mm, vias 2 -> 0
- net Net-(J6-Pad2): track 30.4 -> 20.3 mm
- net Net-(D3-Pad2): track 24.5 -> 32.9 mm
- net Net-(C14-Pad1): track 43.4 -> 36.3 mm

Commit message: updated design
Parts:
- removed J6: STX-3200-3NB, SamacSys_Parts:STX32003NB
- added J1: PH-2W, SHDRRA2W50P0X200_1X2_600X760X510P, F.Cu at (137.6, 70.0)
- J2, J4: value B2B-PH-K-S_LF__SN_ -> PH-2W; footprint SamacSys_Parts:SHDR2W50P0X200_1X2_590X450X600P -> SHDRRA2W50P0X200_1X2_600X760X510P
- J3: value B2B-PH-K-S_LF__SN_ -> WQP-PJ313D; footprint SamacSys_Parts:SHDR2W50P0X200_1X2_590X450X600P -> C18167
- RV1, RV2: value 22k -> 10K_RV; footprint Potentiometer_THT:Potentiometer_Bourns_3296W_Vertical -> 3314J-1
- moved RV2 34.8 mm to (151.8, 85.4), turned to 0 degrees
- moved RV1 32.1 mm to (169.2, 59.8), turned to 180 degrees
- moved J2 29.7 mm to (167.4, 71.8), turned to 270 degrees
- moved J3 20.2 mm to (164.1, 87.4), turned to 180 degrees
- moved R11 7.56 mm to (158.8, 87.4)
- moved J4 1.66 mm to (137.6, 84.2)
Connections:
- AT1 pad 4: 11 -> GND
- C14 pad 2: 11 -> GND
- C17 pad 2: 11 -> GND
- C18 pad 2: 11 -> GND
- C2 pad 2: 11 -> GND
- C3 pad 2: 11 -> GND
- C5 pad 2: 11 -> GND
- D1 pad 2: 11 -> GND
- D2 pad 2: 11 -> GND
- IC1 pad 2: 11 -> GND
- IC1 pad 7: 11 -> GND
- IC2 pad 11: 11 -> (no net)
- J2 pad 1: Net-(D1-Pad1) -> Net-(C14-Pad1)
- J2 pad 2: 11 -> Net-(D3-Pad2)
- J4 pad 2: 11 -> GND
- Q1 pad 2: 11 -> GND
- R11 pad 2: Net-(J6-Pad2) -> Net-(J3-PadA1)
- R14 pad 2: 11 -> GND
- R4 pad 2: 11 -> GND
- R5 pad 2: 11 -> GND
- R7 pad 2: 11 -> GND
- RV1 pad 1: (no net) -> 13
- RV1 pad 2: Net-(R11-Pad1) -> 13
- RV1 pad 3: Net-(C14-Pad1) -> Net-(C13-Pad2)
- RV2 pad 1: 13 -> (no net)
- RV2 pad 2: 13 -> Net-(R11-Pad1)
- RV2 pad 3: Net-(C13-Pad2) -> Net-(C14-Pad1)
- TP2 pad 1: 11 -> GND
Routing:
- net 11: track 143.0 -> 0.00 mm, vias 10 -> 0
- net GND: track 0.00 -> 80.5 mm, vias 0 -> 15
- net Net-(J6-Pad2): track 20.3 -> 0.00 mm
- net Net-(J3-PadA1): track 0.00 -> 8.24 mm
- net +BATT: track 89.7 -> 96.2 mm
- net Net-(C14-Pad1): track 36.3 -> 31.5 mm
- net 13: track 10.9 -> 14.0 mm
- net Net-(C13-Pad2): track 6.02 -> 3.55 mm
- net Net-(R11-Pad1): track 8.08 -> 6.49 mm
- net Net-(D3-Pad2): track 32.9 -> 33.9 mm
- added copper zone on B.Cu, net GND
Other:
- board size 44.2 x 47.2 mm -> 44.2 x 44.8 mm

Commit message: update mfg
Parts:
- renumbered TP1 to BATT, TP2 to GND

Commit message: finished
Parts:
- added JP1: Jumper_2_Bridged, Jumper:SolderJumper-2_P1.3mm_Bridged_Pad1.0x1.5mm, F.Cu at (144.6, 47.6)
- added JP2: Jumper_2_Bridged, Jumper:SolderJumper-2_P1.3mm_Bridged_Pad1.0x1.5mm, F.Cu at (144.6, 53.5)
- added LS1: MLT-7525, MLT7525, F.Cu at (137.1, 50.6)
- J1, J2, J4: value PH-2W -> PH-2V; footprint SHDRRA2W50P0X200_1X2_600X760X510P -> SHDR2W52P0X200_1X2_600X460X630P
- moved J4 32.3 mm to (167.4, 71.8), turned to 270 degrees
- moved J2 29.9 mm to (137.6, 70.0), turned to 90 degrees
- moved J1 14.2 mm to (137.6, 84.2)
- moved C1 4.05 mm to (149.5, 54.3)
- moved AT1 1.96 mm to (147.3, 57.6)
- moved C2 1.96 mm to (152.4, 55.1)
- moved C6 1.96 mm to (152.4, 59.6)
- moved R2 1.96 mm to (152.8, 57.6)
- moved IC3 1.34 mm to (137.3, 60.5)
- moved C3 1.20 mm to (154.9, 57.2)
- moved R4 1.20 mm to (154.9, 59.3)
- renumbered BATT to TP1, GND to TP2
Connections:
- J1 pad 1: Net-(D1-Pad1) -> +BATT
- J2 pad 1: Net-(C14-Pad1) -> Net-(D1-Pad1)
- J2 pad 2: Net-(D3-Pad2) -> GND
- J4 pad 1: +BATT -> Net-(C14-Pad1)
- J4 pad 2: GND -> Net-(D3-Pad2)
Routing:
- net Net-(AT1-Pad2): track 7.25 -> 26.9 mm, vias 0 -> 1
- net Net-(AT1-Pad3): track 9.60 -> 27.6 mm, vias 0 -> 1
- net GND: track 80.5 -> 64.4 mm, vias 15 -> 16
- net +BATT: track 96.2 -> 92.7 mm
- net Net-(JP2-Pad2): track 0.00 -> 3.09 mm
- net Net-(JP1-Pad2): track 0.00 -> 3.06 mm
- net Net-(C6-Pad2): track 7.89 -> 5.53 mm
- net Net-(AT1-Pad8): track 3.36 -> 1.46 mm
- net Net-(AT1-Pad1): track 3.45 -> 5.02 mm
